File: SparkFun_Pro_Micro.sch (KiCad schematic (older format))
At the start: 29 parts, among them P1 USB_C_Plug, U2 MIC5219, U3 ATMEGA32U4, Y1 16MHz

Commit message: nuked everything and reworked decided to work with import from Pro Micro Eagle file.
Parts:
- removed C13, C19: 10uF, Capacitor_Tantalum_SMD:CP_EIA-3216-18_Kemet-A, symbol Device:CP1_Small
- removed D1: Yellow, LED_SMD:LED_0603_1608Metric, symbol Device:LED_Small
- removed D3: Green, LED_SMD:LED_0603_1608Metric, symbol Device:LED_Small
- removed LED1: Red, LED_SMD:LED_0603_1608Metric, symbol Device:LED_Small
- removed R1, R3: 22, Resistor_SMD:R_0603_1608Metric, symbol frmicro-eagle-import:RESISTOR0603-RES
- removed Y1: 16MHz, Crystal:Crystal_SMD_5032-2Pin_5.0x3.2mm, symbol Device:Crystal_Small
- added C13, C19: 10uF, SparkFun_Pro_Micro:EIA3216, symbol SparkFun_Pro_Micro-eagle-import:CAP_POL1206
- added D1: Yellow, SparkFun_Pro_Micro:LED-0603, symbol SparkFun_Pro_Micro-eagle-import:LED0603
- added D3: Green, SparkFun_Pro_Micro:LED-0603, symbol SparkFun_Pro_Micro-eagle-import:LED0603
- added LED1: Red, SparkFun_Pro_Micro:LED-0603, symbol SparkFun_Pro_Micro-eagle-import:LED0603
- added R1, R3: 22, SparkFun_Pro_Micro:0603-RES, symbol SparkFun_Pro_Micro-eagle-import:RESISTOR0603-RES
- added Y1: 16MHz, SparkFun_Pro_Micro:CRYSTAL-SMD-5X3, symbol SparkFun_Pro_Micro-eagle-import:CRYSTAL5X3
- C1, C10, C2, C3, C4, C5, C6: footprint Capacitor_SMD:C_0603_1608Metric -> SparkFun_Pro_Micro:0603-CAP; symbol frmicro-eagle-import:CAP0603-CAP -> SparkFun_Pro_Micro-eagle-import:CAP0603-CAP
- D2: footprint Diode_SMD:D_SOD-323 -> SparkFun_Pro_Micro:SOD-323; symbol frmicro-eagle-import:DIODESOD -> SparkFun_Pro_Micro-eagle-import:DIODESOD
- F1: footprint Fuse:Fuse_1206_3216Metric -> SparkFun_Pro_Micro:PTC-1206; symbol frmicro-eagle-import:PTCSMD -> SparkFun_Pro_Micro-eagle-import:PTCSMD
- JP6, JP7: footprint Connector_PinSocket_2.54mm:PinSocket_1x12_P2.54mm_Vertical -> SparkFun_Pro_Micro:1X12; symbol frmicro-eagle-import:M12PTH -> SparkFun_Pro_Micro-eagle-import:M12PTH
- P1: footprint misc:GCT_USB4155-03-C_REVA -> Connector_USB:USB_C_Plug_Molex_105444
- R11, R2, R4, R5, R6, R7: footprint Resistor_SMD:R_0603_1608Metric -> SparkFun_Pro_Micro:0603-RES; symbol frmicro-eagle-import:RESISTOR0603-RES -> SparkFun_Pro_Micro-eagle-import:RESISTOR0603-RES
- SJ1: footprint Jumper:SolderJumper-2_P1.3mm_Open_Pad1.0x1.5mm -> SparkFun_Pro_Micro:SJ_2S; symbol frmicro-eagle-import:SOLDERJUMPERNC -> SparkFun_Pro_Micro-eagle-import:SOLDERJUMPERNC
- U2: footprint Package_TO_SOT_SMD:SOT-23-5 -> SparkFun_Pro_Micro:SOT23-5; symbol frmicro-eagle-import:V_REG_LDOSMD -> SparkFun_Pro_Micro-eagle-import:V_REG_LDOSMD
- U3: footprint misc:QFN-44-1EP_7x7mm_Pitch0.5mm -> SparkFun_Pro_Micro:QFN-44-NOPAD_1_1-OUTFAKES; symbol frmicro-eagle-import:ATMEGA32U4OUTFAKES -> SparkFun_Pro_Micro-eagle-import:ATMEGA32U4OUTFAKES
Connections:
- wire segments 150 -> 154
Other:
- note added: "Added fuse and diode protection"
- note added: "Added two small squares of tRestrict to keep the ground plane away from the sides of IC legs"
- note added: "Change to 500mA regulator"
- note added: "Changed LEDs to be tied to VCC"
- note added: "Changes on v1.1:"
- note added: "Changes on v1.2:"
- note added: "Changes on v1.3:"
- note added: "Corrected silk on D14"
- note added: "Renamed SS net to D14 (from D17)"
- note added: "Routed directly inward or outward from each leg on the IC"
- note added: "Updated QFN package on 32U4 to be 1:1"
- note added: "Updated package on USB micro B (2 new pads)"
- note added: "Updated symbol of 32U4 in schematic (switched MISO and SS placement)"
- moved on the sheet: R5, R7

Commit message: remove old pro micro schetches
Parts:
- removed C10, C5, C6: 1uF, SparkFun_Pro_Micro:0603-CAP, symbol SparkFun_Pro_Micro-eagle-import:CAP0603-CAP
- removed C13, C19: 10uF, SparkFun_Pro_Micro:EIA3216, symbol SparkFun_Pro_Micro-eagle-import:CAP_POL1206
- removed D2: DIODESOD, SparkFun_Pro_Micro:SOD-323, symbol SparkFun_Pro_Micro-eagle-import:DIODESOD
- removed D3: Green, SparkFun_Pro_Micro:LED-0603, symbol SparkFun_Pro_Micro-eagle-import:LED0603
- removed F1: 500mA, SparkFun_Pro_Micro:PTC-1206, symbol SparkFun_Pro_Micro-eagle-import:PTCSMD
- removed JP6, JP7: M12PTH, SparkFun_Pro_Micro:1X12, symbol SparkFun_Pro_Micro-eagle-import:M12PTH
- removed LED1: Red, SparkFun_Pro_Micro:LED-0603, symbol SparkFun_Pro_Micro-eagle-import:LED0603
- removed P1: USB_C_Plug, Connector_USB:USB_C_Plug_Molex_105444, symbol Connector:USB_C_Plug
- removed R1, R3, R5, R7: 22, SparkFun_Pro_Micro:0603-RES, symbol SparkFun_Pro_Micro-eagle-import:RESISTOR0603-RES
- removed R11: 1K, SparkFun_Pro_Micro:0603-RES, symbol SparkFun_Pro_Micro-eagle-import:RESISTOR0603-RES
- removed R2: 10K, SparkFun_Pro_Micro:0603-RES, symbol SparkFun_Pro_Micro-eagle-import:RESISTOR0603-RES
- removed R4, R6: 330, SparkFun_Pro_Micro:0603-RES, symbol SparkFun_Pro_Micro-eagle-import:RESISTOR0603-RES
- removed SJ1: Closed for 5V Board, SparkFun_Pro_Micro:SJ_2S, symbol SparkFun_Pro_Micro-eagle-import:SOLDERJUMPERNC
- removed U2: MIC5219, SparkFun_Pro_Micro:SOT23-5, symbol SparkFun_Pro_Micro-eagle-import:V_REG_LDOSMD
- removed U3: ATMEGA32U4, SparkFun_Pro_Micro:QFN-44-NOPAD_1_1-OUTFAKES, symbol SparkFun_Pro_Micro-eagle-import:ATMEGA32U4OUTFAKES
- removed Y1: 16MHz, SparkFun_Pro_Micro:CRYSTAL-SMD-5X3, symbol SparkFun_Pro_Micro-eagle-import:CRYSTAL5X3
- added C10, C5, C6: 1.0uF, SparkFun_Pro_Micro:0402-TIGHT, symbol SparkFun_Pro_Micro-eagle-import:1.0UF-0402T-16V-10%
- added C7, C8: 10uF, SparkFun_Pro_Micro:0603, symbol SparkFun_Pro_Micro-eagle-import:10UF-0603-6.3V-20%
- added D2: 3A/10V/280mV, SparkFun_Pro_Micro:SOD-323, symbol SparkFun_Pro_Micro-eagle-import:DIODE-SCHOTTKY-BAT60A
- added D3: GREEN, SparkFun_Pro_Micro:LED-0603, symbol SparkFun_Pro_Micro-eagle-import:LED-GREEN0603
- added F1: 6V 0.5A, SparkFun_Pro_Micro:0805, symbol SparkFun_Pro_Micro-eagle-import:PPTC_6V500MA
- added FRAME1: FRAME-LETTER, SparkFun_Pro_Micro:CREATIVE_COMMONS, symbol SparkFun_Pro_Micro-eagle-import:FRAME-LETTER
- added J3, J4: CONN_12CASTLE, Connector_PinSocket_2.54mm:PinSocket_1x12_P2.54mm_Vertical, symbol SparkFun_Pro_Micro-eagle-import:CONN_12CASTLE
- added J5: USB_C5, Connector_USB:USB_C_Plug_Molex_105444, symbol Connector:USB_C_Plug
- added JP4: JUMPER-SMT_3_1-NC_TRACE_SILK, SparkFun_Pro_Micro:SMT-JUMPER_3_1-NC_TRACE_SILK, symbol SparkFun_Pro_Micro-eagle-import:JUMPER-SMT_3_1-NC_TRACE_SILK
- added LED1: RED, SparkFun_Pro_Micro:LED-0603, symbol SparkFun_Pro_Micro-eagle-import:LED-RED0603
- added LOGO5: SPECIAL_INSTRUCTIONS-ORDERING, SparkFun_Pro_Micro:ORDERING_INSTRUCTIONS, symbol SparkFun_Pro_Micro-eagle-import:SPECIAL_INSTRUCTIONS-ORDERING
- added R1, R3: 5.1k, SparkFun_Pro_Micro:0402-TIGHT, symbol SparkFun_Pro_Micro-eagle-import:5.1KOHM-0402T-1_16W-1%
- added R11, R4, R6: 1k, SparkFun_Pro_Micro:0402-TIGHT, symbol SparkFun_Pro_Micro-eagle-import:1KOHM-0402T-1_16W-1%
- added R2: 10k, SparkFun_Pro_Micro:0402-TIGHT, symbol SparkFun_Pro_Micro-eagle-import:10KOHM-0402T-1_16W-1%
- added R5, R7: 2.2k, SparkFun_Pro_Micro:0402-TIGHT, symbol SparkFun_Pro_Micro-eagle-import:2.2KOHM-0402T-1_16W-1%
- added R8, R9: 22OHM-0402T-1/16W-1%, SparkFun_Pro_Micro:0402-TIGHT, symbol SparkFun_Pro_Micro-eagle-import:22OHM-0402T-1_16W-1%
- added S1: Reset, SparkFun_Pro_Micro:TACTILE_SWITCH_SMD_4.6X2.8MM, symbol SparkFun_Pro_Micro-eagle-import:MOMENTARY-SWITCH-SPST-SMD-4.6X2.8MM
- added U$3: OSHW-LOGOMINI, SparkFun_Pro_Micro:OSHW-LOGO-MINI, symbol SparkFun_Pro_Micro-eagle-import:OSHW-LOGOMINI
- added U1: 3.3V, SparkFun_Pro_Micro:SOT23-5, symbol SparkFun_Pro_Micro-eagle-import:V_REG_AP2112K-3.3V
- added U3: 32U4, SparkFun_Pro_Micro:QFN-44-NOPAD_1_1-LESS_PASTE, symbol SparkFun_Pro_Micro-eagle-import:ATMEGA32U41_1-LESS_PASTE
- added Y2: 16MHz, SparkFun_Pro_Micro:CRYSTAL-SMD-2.0X1.6MM, symbol SparkFun_Pro_Micro-eagle-import:CRYSTAL-16MHZSMD-2X1.6
- C1, C3: footprint SparkFun_Pro_Micro:0603-CAP -> SparkFun_Pro_Micro:0402-TIGHT; symbol SparkFun_Pro_Micro-eagle-import:CAP0603-CAP -> SparkFun_Pro_Micro-eagle-import:0.1UF-0402T-16V-10%
- C2, C4: footprint SparkFun_Pro_Micro:0603-CAP -> SparkFun_Pro_Micro:0402-TIGHT; symbol SparkFun_Pro_Micro-eagle-import:CAP0603-CAP -> SparkFun_Pro_Micro-eagle-import:22PF-0402T-16V-10%
- D1: symbol SparkFun_Pro_Micro-eagle-import:LED0603 -> SparkFun_Pro_Micro-eagle-import:LED-YELLOW0603
Connections:
- net labels added: 3.3V, D2/SDA, D3/SCL, UCAP, V_USB
- net labels removed: A4, A5, D11, D12, D13, D14, D2, D3, UVCC
- wire segments 154 -> 132
- no-connect marks 17 -> 11
Other:
- note added: "32U4 is 5V by default\nI2C Bus is still 3.3V"
- note added: "Arduino Pro Mini Design by Spark Fun Electronics"
- note added: "Max Current Output: 600mA"
- note added: "Max Voltage Input: 6VDC"
- note added: "Microcontroller Voltage Selection"
- note added: "Original Arduino Mini Design by Team Arduino"
- note added: "Pro Micro Design by Spark Fun Electronics"
- note added: "v20"
- note removed: "Added fuse and diode protection"
- note removed: "Added two small squares of tRestrict to keep the ground plane away from the sides of IC legs"
- note removed: "Board is marked with combination of"
- note removed: "Change to 500mA regulator"
- note removed: "Changed LEDs to be tied to VCC"
- note removed: "Changes on v1.1:"
- note removed: "Changes on v1.2:"
- note removed: "Changes on v1.3:"
- note removed: "Corrected silk on D14"
- note removed: "Max Current Output: 500mA"
- note removed: "Max Voltage Input: 16VDC"
- note removed: "Not used"
- note removed: "Open for 3.3V Board"
- note removed: "Renamed SS net to D14 (from D17)"
- note removed: "Routed directly inward or outward from each leg on the IC"
- note removed: "Updated QFN package on 32U4 to be 1:1"
- note removed: "Updated package on USB micro B (2 new pads)"
- note removed: "Updated symbol of 32U4 in schematic (switched MISO and SS placement)"
- note removed: "VCC = 5V or 3.3V Output"
- note removed: "resonator frequency and regulator voltage."
- moved on the sheet: C1, C2, C3, C4
